Commit message: [hironx_tutorial] Adjust odom for HIRONXJSK

File: hironx_tutorial/models/HIRONXJSK.gazebo.xacro (robot description, xacro)
@@ -11,5 +11,5 @@
   <link name="odom" />
   <joint name="odom_to_WAIST_Link" type="fixed">
-    <origin rpy="0 0 0" xyz="0 0.0 0.97" />
+    <origin rpy="0 0 0" xyz="0 0.0 0.80" />
     <parent link="odom" />
     <child link="WAIST_Link" />

Commit message: [hironx_tutorial] Fix WAIST_Link -> WAIST

File: hironx_tutorial/models/HIRONXJSK.gazebo.xacro (robot description, xacro)
@@ -10,8 +10,8 @@
   </gazebo>
   <link name="odom" />
-  <joint name="odom_to_WAIST_Link" type="fixed">
+  <joint name="odom_to_WAIST" type="fixed">
     <origin rpy="0 0 0" xyz="0 0.0 0.80" />
     <parent link="odom" />
-    <child link="WAIST_Link" />
+    <child link="WAIST" />
   </joint>
   <!-- copied from   fetch_description/robots/fetch.urdf -->

Commit message: [hironx_tutorial] Fix HIRONXJSK to gazebo world

File: hironx_tutorial/models/HIRONXJSK.gazebo.xacro (robot description, xacro)
@@ -14,4 +14,10 @@
     <parent link="odom" />
     <child link="WAIST" />
+  </joint>
+  <!-- Fix robot to Gazebo world with 'odom' frame -->
+  <link name="world" />
+  <joint name="fixed" type="fixed">
+    <parent link="world" />
+    <child link="odom" />
   </joint>
   <!-- copied from   fetch_description/robots/fetch.urdf -->

Commit message: [hironx_tutorial] Fix camera links of HIRONXJSK

File: hironx_tutorial/models/HIRONXJSK.gazebo.xacro (robot description, xacro)
@@ -21,8 +21,8 @@
     <child link="odom" />
   </joint>
-  <!-- copied from   fetch_description/robots/fetch.urdf -->
+  <!-- Based on fetch_description/robots/fetch.urdf -->
   <link name="head_camera_rgb_frame" />
   <joint name="head_camera_rgb_joint" type="fixed">
-    <origin rpy="0 0 0" xyz="0 0.02 0" />
+    <origin rpy="0 0 0" xyz="0.057 0.02 0.1" />
     <parent link="HEAD_JOINT1_Link" />
     <child link="head_camera_rgb_frame" />
@@ -36,5 +36,5 @@
   <link name="head_camera_depth_frame" />
   <joint name="head_camera_depth_joint" type="fixed">
-    <origin rpy="0 0 0" xyz="0 0.045 0" />
+    <origin rpy="0 0 0" xyz="0.057 0.045 0.1" />
     <parent link="HEAD_JOINT1_Link" />
     <child link="head_camera_depth_frame" />

Commit message: [hironx_tutorial] Stop fixing robot to 'world'
See https://github.com/tork-a/rtmros_nextage/issues/235#issuecomment-619514563

File: hironx_tutorial/models/HIRONXJSK.gazebo.xacro (robot description, xacro)
@@ -14,10 +14,4 @@
     <parent link="odom" />
     <child link="WAIST" />
-  </joint>
-  <!-- Fix robot to Gazebo world with 'odom' frame -->
-  <link name="world" />
-  <joint name="fixed" type="fixed">
-    <parent link="world" />
-    <child link="odom" />
   </joint>
   <!-- Based on fetch_description/robots/fetch.urdf -->

Commit message: [hironx_tutorial] Stop converting HIRONXJSK model
It is executed at hrpsys_ros_bridge_tutorials layer

File: hironx_tutorial/models/HIRONXJSK.gazebo.xacro (robot description, xacro)
@@ -1,5 +1,5 @@
 <?xml version="1.0"?>
 <robot name="HIRONXJSK" xmlns:xacro="http://www.ros.org/wiki/xacro">
-  <xacro:include filename="$(find hironx_tutorial)/models/HIRONXJSK.urdf" />
+  <xacro:include filename="$(find hrpsys_ros_bridge_tutorials)/models/HIRONXJSK_SENSORS.urdf" />
   <!-- Gazebo plugin for ROS Control -->
   <gazebo>
@@ -14,29 +14,4 @@
     <parent link="odom" />
     <child link="WAIST" />
-  </joint>
-  <!-- Based on fetch_description/robots/fetch.urdf -->
-  <link name="head_camera_rgb_frame" />
-  <joint name="head_camera_rgb_joint" type="fixed">
-    <origin rpy="0 0 0" xyz="0.057 0.02 0.1" />
-    <parent link="HEAD_JOINT1_Link" />
-    <child link="head_camera_rgb_frame" />
-  </joint>
-  <link name="head_camera_rgb_optical_frame" />
-  <joint name="head_camera_rgb_optical_joint" type="fixed">
-    <origin rpy="-1.57079632679 0 -1.57079632679" xyz="0 0 0" />
-    <parent link="head_camera_rgb_frame" />
-    <child link="head_camera_rgb_optical_frame" />
-  </joint>
-  <link name="head_camera_depth_frame" />
-  <joint name="head_camera_depth_joint" type="fixed">
-    <origin rpy="0 0 0" xyz="0.057 0.045 0.1" />
-    <parent link="HEAD_JOINT1_Link" />
-    <child link="head_camera_depth_frame" />
-  </joint>
-  <link name="head_camera_depth_optical_frame" />
-  <joint name="head_camera_depth_optical_joint" type="fixed">
-    <origin rpy="-1.57079632679 0 -1.57079632679" xyz="0 0 0" />
-    <parent link="head_camera_depth_frame" />
-    <child link="head_camera_depth_optical_frame" />
   </joint>
   <!-- copied from fetch_gazebo/robots/fetch.gazebo.xacro -->
